File: scheme/aquarium_touch/aquarium_touch.kicad_sch (KiCad schematic)
At the start: 12 parts, among them J1 Conn_01x06_Socket, J2 E201-BNC, K1 Relay_SPDT, Q1 BC547

Commit message: Salvataggio del 17/10/2026  9:22:35,08
Connections:
- net at DS18B20.1 (Pin_1), R3.1: now also LIGHT1.2 (Pin_2)
- net at R3.2: now also R4.1; no longer LIGHT1.2 (Pin_2)
Changed lines of the file:
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@@
 	(text "R3 20kΩ"
 		(exclude_from_sim no)
-		(at 172.72 35.56 0)
+		(at 176.53 35.56 0)
 		(effects
 			(font
@@
 	)
 	(junction
+		(at 162.56 43.18)
+		(diameter 0)
+		(color 0 0 0 1)
+	)
+	(junction
 		(at 172.72 74.93)
 		(diameter 0)
@@
 	)
 	(junction
+		(at 180.34 30.48)
+		(diameter 0)
+		(color 255 229 191 1)
+	)
+	(junction
 		(at 163.83 72.39)
 		(diameter 0)
@@
 	)
 	(junction
-		(at 162.56 43.18)
-		(diameter 0)
-		(color 0 0 0 1)
-	)
-	(junction
 		(at 180.34 74.93)
 		(diameter 0)
@@
 		(color 0 0 0 0)
 	)
-	(wire
-		(pts
-			(xy 162.56 33.02) (xy 168.91 33.02)
-		)
-		(stroke
-			(width 0)
-			(type default)
-			(color 0 0 0 1)
-		)
+	(junction
+		(at 162.56 36.83)
+		(diameter 0)
+		(color 0 0 0 1)
 	)
 	(wire
@@
 	(wire
 		(pts
+			(xy 180.34 30.48) (xy 160.02 30.48)
+		)
+		(stroke
+			(width 0)
+			(type default)
+			(color 255 229 191 1)
+		)
+	)
+	(wire
+		(pts
 			(xy 210.82 35.56) (xy 210.82 67.31)
 		)
@@
 	(wire
 		(pts
+			(xy 162.56 43.18) (xy 162.56 36.83)
+		)
+		(stroke
+			(width 0)
+			(type default)
+			(color 0 0 0 1)
+		)
+	)
+	(wire
+		(pts
 			(xy 186.69 50.8) (xy 189.23 50.8)
 		)
@@
 	(wire
 		(pts
+			(xy 162.56 33.02) (xy 162.56 36.83)
+		)
+		(stroke
+			(width 0)
+			(type default)
+			(color 0 0 0 1)
+		)
+	)
+	(wire
+		(pts
 			(xy 156.21 95.25) (xy 162.56 95.25)
 		)
@@
 	(wire
 		(pts
+			(xy 208.28 33.02) (xy 222.25 33.02)
+		)
+		(stroke
+			(width 0)
+			(type default)
+			(color 0 0 0 1)
+		)
+	)
+	(wire
+		(pts
 			(xy 207.01 102.87) (xy 213.36 102.87)
 		)
@@
 	(wire
 		(pts
+			(xy 208.28 36.83) (xy 208.28 33.02)
+		)
+		(stroke
+			(width 0)
+			(type default)
+			(color 0 0 0 1)
+		)
+	)
+	(wire
+		(pts
 			(xy 189.23 58.42) (xy 189.23 67.31)
 		)
@@
 	(wire
 		(pts
-			(xy 50.8 177.8) (xy 124.46 177.8)
+			(xy 162.56 36.83) (xy 208.28 36.83)
 		)
 		(stroke
 			(width 0)
 			(type default)
-			(color 0 255 255 1)
+			(color 0 0 0 1)
 		)
 	)
 	(wire
 		(pts
-			(xy 48.26 180.34) (xy 127 180.34)
+			(xy 50.8 177.8) (xy 124.46 177.8)
 		)
 		(stroke
 			(width 0)
 			(type default)
-			(color 255 0 0 1)
+			(color 0 255 255 1)
 		)
 	)
 	(wire
 		(pts
-			(xy 162.56 33.02) (xy 162.56 43.18)
+			(xy 48.26 180.34) (xy 127 180.34)
 		)
 		(stroke
 			(width 0)
 			(type default)
-			(color 0 0 0 1)
+			(color 255 0 0 1)
 		)
 	)
@@
 	(wire
 		(pts
-			(xy 176.53 33.02) (xy 222.25 33.02)
+			(xy 180.34 74.93) (xy 222.25 74.93)
 		)
 		(stroke
 			(width 0)
 			(type default)
-			(color 0 0 0 1)
+			(color 255 153 0 1)
 		)
 	)
 	(wire
 		(pts
-			(xy 180.34 74.93) (xy 222.25 74.93)
+			(xy 127 180.34) (xy 127 102.87)
 		)
 		(stroke
 			(width 0)
 			(type default)
-			(color 255 153 0 1)
+			(color 255 0 0 1)
 		)
 	)
 	(wire
 		(pts
-			(xy 127 180.34) (xy 127 102.87)
+			(xy 48.26 163.83) (xy 48.26 180.34)
 		)
 		(stroke
@@
 	(wire
 		(pts
-			(xy 48.26 163.83) (xy 48.26 180.34)
+			(xy 172.72 33.02) (xy 162.56 33.02)
 		)
 		(stroke
 			(width 0)
 			(type default)
-			(color 255 0 0 1)
+			(color 0 0 0 1)
 		)
 	)
@@
 	(wire
 		(pts
+			(xy 180.34 30.48) (xy 180.34 33.02)
+		)
+		(stroke
+			(width 0)
+			(type default)
+			(color 255 229 191 1)
+		)
+	)
+	(wire
+		(pts
 			(xy 171.45 63.5) (xy 172.72 63.5)
 		)
@@
 	(wire
 		(pts
-			(xy 181.61 30.48) (xy 160.02 30.48)
+			(xy 181.61 30.48) (xy 180.34 30.48)
 		)
 		(stroke
@@
 	(symbol
 		(lib_id "Device:R")
-		(at 172.72 33.02 90)
+		(at 176.53 33.02 90)
 		(unit 1)
 		(body_style 1)
@@
 		(fields_autoplaced yes)
 		(property "Reference" "R3"
-			(at 171.4499 30.48 0)
+			(at 175.2599 30.48 0)
 			(hide yes)
 			(show_name no)
@@
 		)
 		(property "Value" "R"
-			(at 173.9899 30.48 0)
+			(at 177.7999 30.48 0)
 			(hide yes)
 			(show_name no)
@@
 		)
 		(property "Footprint" ""
-			(at 172.72 34.798 90)
+			(at 176.53 34.798 90)
 			(hide yes)
 			(show_name no)
@@
 		)
 		(property "Datasheet" ""
-			(at 172.72 33.02 0)
+			(at 176.53 33.02 0)
 			(hide yes)
 			(show_name no)
@@
 		)
 		(property "Description" "Resistor"
-			(at 172.72 33.02 0)
+			(at 176.53 33.02 0)
 			(hide yes)
 			(show_name no)
